File: _autosave-stm32_devboard.kicad_pcb (KiCad board)
At the start: 2 copper layers, 46 parts, among them J1 Conn_01x04_Male, J2 USB_B_Micro, J3 Micro_SD_Card, J4 Conn_01x05_Male, SW1 SW_SPDT, U1 NCP5501DT33RKG, U2 STM32F103CBT6, U3 LSM303C, Y1 Crystal_GND24

Commit message: layout and sch update
Parts:
- moved C13 0.66 mm to (85.0, 99.1), turned to 180 degrees
Changed lines of the file:
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@@
   )
   (footprint "Capacitor_SMD:C_0603_1608Metric" (layer "F.Cu")
-    (at 84.4 99.2 -90)
+    (at 85.05 99.1 180)
     (descr "Capacitor SMD 0603 (1608 Metric), square (rectangular) end terminal, IPC_7351 nominal, (Body size source: IPC-SM-782 page 76, https://www.pcb-3d.com/wordpress/wp-content/uploads/ipc-sm-782a_amendment_1_and_2.pdf), generated with kicad-footprint-generator")
     (tags "capacitor")
@@
     (property "Sheetname" "")
     (attr smd)
-    (fp_text reference "C13" (at 2.5 0.25 180) (layer "F.SilkS")
+    (fp_text reference "C13" (at 0.15 -1.6 180) (layer "F.SilkS")
       (effects (font (size 1 1) (thickness 0.15)))
     )
-    (fp_text value "10u" (at 0 1.43 90) (layer "F.Fab")
+    (fp_text value "10u" (at 0 1.43) (layer "F.Fab")
       (effects (font (size 1 1) (thickness 0.15)))
     )
-    (fp_text user "${REFERENCE}" (at 0 0 90) (layer "F.Fab")
+    (fp_text user "${REFERENCE}" (at 0 0) (layer "F.Fab")
       (effects (font (size 0.4 0.4) (thickness 0.06)))
     )
@@
     (fp_line (start -0.8 0.4) (end -0.8 -0.4) (layer "F.Fab") (width 0.1))
     (fp_line (start 0.8 -0.4) (end 0.8 0.4) (layer "F.Fab") (width 0.1))
-    (pad "1" smd roundrect locked (at -0.775 0 270) (size 0.9 0.95) (layers "F.Cu" "F.Paste" "F.Mask") (roundrect_rratio 0.25)
+    (pad "1" smd roundrect locked (at -0.775 0 180) (size 0.9 0.95) (layers "F.Cu" "F.Paste" "F.Mask") (roundrect_rratio 0.25)
       (net 7 "VBUS") (pintype "passive"))
-    (pad "2" smd roundrect locked (at 0.775 0 270) (size 0.9 0.95) (layers "F.Cu" "F.Paste" "F.Mask") (roundrect_rratio 0.25)
+    (pad "2" smd roundrect locked (at 0.775 0 180) (size 0.9 0.95) (layers "F.Cu" "F.Paste" "F.Mask") (roundrect_rratio 0.25)
       (net 2 "GND") (pintype "passive"))
     (model "${KICAD6_3DMODEL_DIR}/Capacitor_SMD.3dshapes/C_0603_1608Metric.wrl"
