File: _autosave-stm32_devboard.kicad_sch (KiCad schematic)
At the start: 46 parts, among them J1 Conn_01x04_Male, J2 USB_B_Micro, J3 Micro_SD_Card, J4 Conn_01x05_Male, SW1 SW_SPDT, U1 NCP5501DT33RKG, U2 STM32F103CBT6, U3 LSM303C, Y1 Crystal_GND24

Commit message: layout and sch update
Changed lines of the file:
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@@
   (symbol (lib_id "power:+3.3V") (at 173.99 81.28 0) (unit 1)
     (in_bom yes) (on_board yes)
-    (property "Reference" "#PWR?" (id 0) (at 173.99 85.09 0)
+    (property "Reference" "#PWR0117" (id 0) (at 173.99 85.09 0)
       (effects (font (size 1.27 1.27)) hide)
     )
@@
   )
   (symbol (lib_id "power:GND") (at 173.99 91.44 0) (unit 1)
-    (in_bom yes) (on_board yes) (fields_autoplaced)
-    (property "Reference" "#PWR?" (id 0) (at 173.99 97.79 0)
-      (effects (font (size 1.27 1.27)) hide)
-    )
-    (property "Value" "GND" (id 1) (at 173.99 96.52 0))
+    (in_bom yes) (on_board yes)
+    (property "Reference" "#PWR0118" (id 0) (at 173.99 97.79 0)
+      (effects (font (size 1.27 1.27)) hide)
+    )
+    (property "Value" "GND" (id 1) (at 176.53 91.44 0))
     (property "Footprint" "" (id 2) (at 173.99 91.44 0)
       (effects (font (size 1.27 1.27)) hide)
@@
     )
     (path "/01160f7c-6c3b-4f8a-a6b1-d2edd70e4083"
-      (reference "#PWR?") (unit 1) (value "+3.3V") (footprint "")
+      (reference "#PWR0117") (unit 1) (value "+3.3V") (footprint "")
     )
     (path "/b6740d20-5f29-48ad-b5ce-1521e5e5040d"
-      (reference "#PWR?") (unit 1) (value "GND") (footprint "")
+      (reference "#PWR0118") (unit 1) (value "GND") (footprint "")
     )
     (path "/7fcf6ddc-297f-4c92-867e-65041a6dad67"
