File: _autosave-stm32_devboard.kicad_sch (KiCad schematic)
At the start: 50 parts, among them J1 Conn_01x04_Male, J2 USB_B_Micro, J3 Micro_SD_Card, J4 Conn_01x05_Male, SW1 SW_SPDT, U1 NCP5501DT33RKG, U2 STM32F103CBT6, U3 LSM303C, Y1 Crystal_GND24

Commit message: finish
Parts:
- gave numbers to parts that had none: 4
Changed lines of the file:
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@@
   (symbol (lib_id "Mechanical:MountingHole") (at 198.12 151.13 0) (unit 1)
     (in_bom yes) (on_board yes) (fields_autoplaced)
-    (property "Reference" "H?" (id 0) (at 200.66 149.8599 0)
+    (property "Reference" "H1" (id 0) (at 200.66 149.8599 0)
       (effects (font (size 1.27 1.27)) (justify left))
     )
@@
   (symbol (lib_id "Mechanical:MountingHole") (at 198.12 156.21 0) (unit 1)
     (in_bom yes) (on_board yes) (fields_autoplaced)
-    (property "Reference" "H?" (id 0) (at 200.66 154.9399 0)
+    (property "Reference" "H2" (id 0) (at 200.66 154.9399 0)
       (effects (font (size 1.27 1.27)) (justify left))
     )
@@
   (symbol (lib_id "Mechanical:MountingHole") (at 218.44 151.13 0) (unit 1)
     (in_bom yes) (on_board yes) (fields_autoplaced)
-    (property "Reference" "H?" (id 0) (at 220.98 149.8599 0)
+    (property "Reference" "H3" (id 0) (at 220.98 149.8599 0)
       (effects (font (size 1.27 1.27)) (justify left))
     )
@@
   (symbol (lib_id "Mechanical:MountingHole") (at 219.71 157.48 0) (unit 1)
     (in_bom yes) (on_board yes) (fields_autoplaced)
-    (property "Reference" "H?" (id 0) (at 222.25 156.2099 0)
+    (property "Reference" "H4" (id 0) (at 222.25 156.2099 0)
       (effects (font (size 1.27 1.27)) (justify left))
     )
@@
     )
     (path "/6791df4a-e5fd-44fc-8069-1df8ab313ee3"
-      (reference "H?") (unit 1) (value "MountingHole") (footprint "MountingHole:MountingHole_2.2mm_M2")
+      (reference "H1") (unit 1) (value "MountingHole") (footprint "MountingHole:MountingHole_2.2mm_M2")
     )
     (path "/c6e080f2-c535-4467-98bf-40ee712b30f3"
-      (reference "H?") (unit 1) (value "MountingHole") (footprint "MountingHole:MountingHole_2.2mm_M2")
+      (reference "H2") (unit 1) (value "MountingHole") (footprint "MountingHole:MountingHole_2.2mm_M2")
     )
     (path "/d710793d-17d0-4ec0-8141-38b711e11f68"
-      (reference "H?") (unit 1) (value "MountingHole") (footprint "MountingHole:MountingHole_2.2mm_M2")
+      (reference "H3") (unit 1) (value "MountingHole") (footprint "MountingHole:MountingHole_2.2mm_M2")
     )
     (path "/dd9ad22d-d55a-40b2-9e09-890b28829832"
-      (reference "H?") (unit 1) (value "MountingHole") (footprint "MountingHole:MountingHole_2.2mm_M2")
+      (reference "H4") (unit 1) (value "MountingHole") (footprint "MountingHole:MountingHole_2.2mm_M2")
     )
     (path "/eaa5ff37-3211-499b-b611-26b2603edc6a"
