File: stm32_devboard.kicad_pcb (KiCad board)
At the start: 2 copper layers, 46 parts, among them J1 Conn_01x04_Male, J2 USB_B_Micro, J3 Micro_SD_Card, J4 Conn_01x05_Male, SW1 SW_SPDT, U1 NCP5501DT33RKG, U2 STM32F103CBT6, U3 LSM303C, Y1 Crystal_GND24

Commit message: finish
Parts:
- added H1: MountingHole, MountingHole:MountingHole_2.2mm_M2, F.Cu at (168.3, 66.8)
- added H2: MountingHole, MountingHole:MountingHole_2.2mm_M2, F.Cu at (202.4, 102.9)
- added H3: MountingHole, MountingHole:MountingHole_2.2mm_M2, F.Cu at (202.4, 66.8)
- added H4: MountingHole, MountingHole:MountingHole_2.2mm_M2, F.Cu at (168.3, 102.8)
- moved C3 118.5 mm to (185.7, 72.2), turned to 180 degrees
- moved C2 114.0 mm to (180.8, 78.2)
- moved C4 113.9 mm to (180.7, 80.4)
- moved Y1 113.3 mm to (177.7, 79.3)
- moved J4 112.8 mm to (184.0, 103.4)
- moved D1 112.7 mm to (195.0, 94.9), turned to -90 degrees
- moved J2 112.6 mm to (201.8, 77.9)
- moved J3 112.6 mm to (171.4, 91.3)
- moved C7 112.5 mm to (191.7, 85.2)
- moved D5 112.5 mm to (189.1, 88.9)
- moved C19 112.4 mm to (177.2, 72.4), turned to 90 degrees
- moved C13 112.4 mm to (195.8, 80.4)
- moved C17 112.4 mm to (177.1, 68.2)
- moved C18 112.4 mm to (175.3, 69.7)
- moved C8 112.4 mm to (182.5, 77.1)
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Connections:
- U3 pad 12: /INT_ACCEL -> /INT_XL
Routing:
- net +3V3: track 0.00 -> 234.4 mm, vias 0 -> 14
- net GND: track 0.00 -> 61.3 mm, vias 0 -> 31
- net /SD_VDD: track 0.00 -> 42.1 mm, vias 0 -> 4
- net IMU_SDA: track 0.00 -> 38.9 mm
- net SD_MISO: track 0.00 -> 38.2 mm
- net /INT_MAG: track 0.00 -> 32.9 mm, vias 0 -> 2
- net SD_MOSI: track 0.00 -> 30.6 mm, vias 0 -> 4
- net SD_SS: track 0.00 -> 24.1 mm, vias 0 -> 2
- net SD_SCK: track 0.00 -> 23.4 mm
- net /GPIO_1: track 0.00 -> 22.5 mm
- net /GPIO_2: track 0.00 -> 21.7 mm
- net /GPIO_3: track 0.00 -> 21.0 mm
- net IMU_SCL: track 0.00 -> 18.2 mm
- net /INT_XL: track 0.00 -> 16.9 mm, vias 0 -> 2
- net /SW_BOOT0: track 0.00 -> 14.0 mm
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- added copper zone on F.Cu, net +3V3
- added copper zone on B.Cu, net GND
- added copper zone on F.Cu, net GND
- added copper zone on F.Cu, net VBUS
Other:
- board outline added: 40.9 x 42.8 mm

Commit message: Update stm32_devboard.kicad_pcb
Parts:
- moved C14 0.38 mm to (189.0, 93.9)
Routing:
- net +3V3: track 234.4 -> 238.0 mm
- net /INT_XL: track 16.9 -> 17.6 mm
- net /INT_MAG: track 32.9 -> 33.4 mm
